Commit message: add controller

File: robots/rsc_car.urdf (robot description, URDF)
Before this commit: robot rsc_car, 4 links, 3 joints
Links:
- added link base_footprint; visual box size=0 0 0
Joints:
- added joint base_footprint_joint: type fixed, parent base_footprint, child base_link, origin xyz=0 0.00594553148142892 0 rpy=0 0 0
- joint rwheel_joint: axis 0 -1 0 -> 0 1 0

Commit message: completed

File: robots/rsc_car.urdf (robot description, URDF)
Before this commit: robot rsc_car, 5 links, 4 joints
Joints:
- joint base_footprint_joint: origin xyz=0 0.00594553148142892 0 rpy=0 0 0 -> xyz=0 0 0.1124430740677247 rpy=0 0 0

Commit message: add install flags in CMakeLists.txt

File: robots/rsc_car.urdf (robot description, URDF)
Before this commit: robot rsc_car, 5 links, 4 joints
Links:
- link base_link: geometry collision mesh filename=package://rsc_car_description/meshes/base_link.STL; visual mesh filename=package://rsc_car_description/meshes/base_link.STL
- link hokuyo_link: geometry collision mesh filename=package://rsc_car_description/meshes/hokuyo_link.STL; visual mesh filename=package://rsc_car_description/meshes/hokuyo_link.STL
- link lwheel_link: geometry collision mesh filename=package://rsc_car_description/meshes/lwheel_link.STL; visual mesh filename=package://rsc_car_description/meshes/lwheel_link.STL
- link rwheel_link: geometry collision mesh filename=package://rsc_car_description/meshes/rwheel_link.STL; visual mesh filename=package://rsc_car_description/meshes/rwheel_link.STL
